File: hardware/breakout/breakout.brd (EAGLE design)
At the start: 30 x 35.3 mm, 20 parts, among them J3 IMPULSE_GECKO_HEADER, J4 SPRING-TERMINAL_3/PTSA-ZZ_2.5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, J5 SPRING-TERMINAL_3/PTSA-ZZ_2.5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, J6 SPRING-TERMINAL_2/PTSA-ZZ_2.5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, J7 SPRING-TERMINAL_2/PTSA-ZZ_2.5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

Commit message: updates to boards
Other:
- board text added: "2013/10/11"
- board text removed: "2013/ 10/11"
