File: hardware/buzz/rev_a/buzz.sch (EAGLE design)
At the start: 5 parts, among them J1 IMPULSE_GECKO_HEADER, X1 MSP1007, X2 MSP1007

Commit message: updates to boards
Parts:
- added TP1: TEST_POINT_0.040IN, headers:TEST_POINT_0.040IN
Connections:
- net TRIGGER: now also TP1.TESTPOINT
Changed lines of the file:
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@@
 <part name="X2" library="activator" deviceset="MSP1007" device=""/>
 <part name="U$3" library="logos" deviceset="UMICH_SOLID" device="_SMALL+"/>
+<part name="TP1" library="headers" deviceset="TEST_POINT_0.040IN" device=""/>
 </parts>
 <sheets>
@@
 <instance part="X2" gate="G$1" x="50.8" y="104.14" rot="R180"/>
 <instance part="U$3" gate="G$1" x="231.14" y="172.72"/>
+<instance part="TP1" gate="G$1" x="104.14" y="96.52" rot="R270"/>
 </instances>
 <busses>
@@
 <segment>
 <pinref part="D1" gate="G$1" pin="A"/>
-<wire x1="101.6" y1="88.9" x2="106.68" y2="88.9" width="0.1524" layer="91"/>
+<wire x1="101.6" y1="88.9" x2="104.14" y2="88.9" width="0.1524" layer="91"/>
 <label x="106.68" y="88.9" size="1.27" layer="95" xref="yes"/>
+<pinref part="TP1" gate="G$1" pin="TESTPOINT"/>
+<wire x1="104.14" y1="88.9" x2="106.68" y2="88.9" width="0.1524" layer="91"/>
+<wire x1="104.14" y1="93.98" x2="104.14" y2="88.9" width="0.1524" layer="91"/>
+<junction x="104.14" y="88.9"/>
 </segment>
 </net>
